Commit message: color works

File: solo_legged_gym/resources/robots/solo12/urdf/solo12.urdf (robot description, URDF)
Before this commit: robot solo, 17 links, 16 joints
Joints:
- joint FL_HAA: limit lower=-3.14159265359 upper=3.14159265359 effort=1000 velocity=30 -> lower=-1.0471975512 upper=1.0471975512 effort=1000 velocity=30
- joint FL_HFE: limit lower=-3.14159265359 upper=3.14159265359 effort=1000 velocity=30 -> lower=0.0 upper=1.57079632679 effort=1000 velocity=30
- joint FL_KFE: limit lower=-3.14159265359 upper=3.14159265359 effort=1000 velocity=30 -> lower=-3.14159265359 upper=0.0 effort=1000 velocity=30
- joint FR_HAA: limit lower=-3.14159265359 upper=3.14159265359 effort=1000 velocity=30 -> lower=-1.0471975512 upper=1.0471975512 effort=1000 velocity=30
- joint FR_HFE: limit lower=-3.14159265359 upper=3.14159265359 effort=1000 velocity=30 -> lower=0.0 upper=1.57079632679 effort=1000 velocity=30
- joint FR_KFE: limit lower=-3.14159265359 upper=3.14159265359 effort=1000 velocity=30 -> lower=-3.14159265359 upper=0.0 effort=1000 velocity=30
- joint HL_HAA: limit lower=-3.14159265359 upper=3.14159265359 effort=1000 velocity=30 -> lower=-1.0471975512 upper=1.0471975512 effort=1000 velocity=30
- joint HL_HFE: limit lower=-3.14159265359 upper=3.14159265359 effort=1000 velocity=30 -> lower=-1.57079632679 upper=0.0 effort=1000 velocity=30
- joint HL_KFE: limit lower=-3.14159265359 upper=3.14159265359 effort=1000 velocity=30 -> lower=0.0 upper=3.14159265359 effort=1000 velocity=30
- joint HR_HAA: limit lower=-3.14159265359 upper=3.14159265359 effort=1000 velocity=30 -> lower=-1.0471975512 upper=1.0471975512 effort=1000 velocity=30
- joint HR_HFE: limit lower=-3.14159265359 upper=3.14159265359 effort=1000 velocity=30 -> lower=-1.57079632679 upper=0.0 effort=1000 velocity=30
- joint HR_KFE: limit lower=-3.14159265359 upper=3.14159265359 effort=1000 velocity=30 -> lower=0.0 upper=3.14159265359 effort=1000 velocity=30

Commit message: WIP

File: solo_legged_gym/resources/robots/solo12/urdf/solo12.urdf (robot description, URDF)
Before this commit: robot solo, 17 links, 16 joints
Joints:
- joint FL_HAA: limit lower=-1.0471975512 upper=1.0471975512 effort=1000 velocity=30 -> lower=-1.57079632679 upper=1.57079632679 effort=1000 velocity=30
- joint FL_HFE: limit lower=0.0 upper=1.57079632679 effort=1000 velocity=30 -> lower=-1.57079632679 upper=1.57079632679 effort=1000 velocity=30
- joint FL_KFE: limit lower=-3.14159265359 upper=0.0 effort=1000 velocity=30 -> lower=-3.14159265359 upper=3.14159265359 effort=1000 velocity=30
- joint FR_HAA: limit lower=-1.0471975512 upper=1.0471975512 effort=1000 velocity=30 -> lower=-1.57079632679 upper=1.57079632679 effort=1000 velocity=30
- joint FR_HFE: limit lower=0.0 upper=1.57079632679 effort=1000 velocity=30 -> lower=-1.57079632679 upper=1.57079632679 effort=1000 velocity=30
- joint FR_KFE: limit lower=-3.14159265359 upper=0.0 effort=1000 velocity=30 -> lower=-3.14159265359 upper=3.14159265359 effort=1000 velocity=30
- joint HL_HAA: limit lower=-1.0471975512 upper=1.0471975512 effort=1000 velocity=30 -> lower=-1.57079632679 upper=1.57079632679 effort=1000 velocity=30
- joint HL_HFE: limit lower=-1.57079632679 upper=0.0 effort=1000 velocity=30 -> lower=-1.57079632679 upper=1.57079632679 effort=1000 velocity=30
- joint HL_KFE: limit lower=0.0 upper=3.14159265359 effort=1000 velocity=30 -> lower=-3.14159265359 upper=3.14159265359 effort=1000 velocity=30
- joint HR_HAA: limit lower=-1.0471975512 upper=1.0471975512 effort=1000 velocity=30 -> lower=-1.57079632679 upper=1.57079632679 effort=1000 velocity=30
- joint HR_HFE: limit lower=-1.57079632679 upper=0.0 effort=1000 velocity=30 -> lower=-1.57079632679 upper=1.57079632679 effort=1000 velocity=30
- joint HR_KFE: limit lower=0.0 upper=3.14159265359 effort=1000 velocity=30 -> lower=-3.14159265359 upper=3.14159265359 effort=1000 velocity=30

Commit message: WIP

File: solo_legged_gym/resources/robots/solo12/urdf/solo12.urdf (robot description, URDF)
Before this commit: robot solo, 17 links, 16 joints
Joints:
- joint FL_HAA: limit lower=-1.57079632679 upper=1.57079632679 effort=1000 velocity=30 -> lower=-1.0471975512 upper=1.0471975512 effort=1000 velocity=30
- joint FR_HAA: limit lower=-1.57079632679 upper=1.57079632679 effort=1000 velocity=30 -> lower=-1.0471975512 upper=1.0471975512 effort=1000 velocity=30
- joint HL_HAA: limit lower=-1.57079632679 upper=1.57079632679 effort=1000 velocity=30 -> lower=-1.0471975512 upper=1.0471975512 effort=1000 velocity=30
- joint HR_HAA: limit lower=-1.57079632679 upper=1.57079632679 effort=1000 velocity=30 -> lower=-1.0471975512 upper=1.0471975512 effort=1000 velocity=30
